Commit message: imu.integrated

File: rc_map/urdf/waking_robot.xacro (robot description, xacro)
@@ -11,21 +11,4 @@
         </inertial>
     </xacro:macro>
-    <link name="base_footprint">
-        <visual>
-            <geometry>
-                <box size="0.001 0.001 0.001"/>
-            </geometry>
-            <origin rpy="0 0 0" xyz="0 0 0"/>
-        </visual>
-    </link>
-    <gazebo reference="base_footprint">
-        <material>Gazebo/Green</material>
-        <turnGravityOff>false</turnGravityOff>
-    </gazebo>
-    <joint name="base_footprint_joint" type="fixed">
-        <origin xyz="0 0 0" />
-        <parent link="base_footprint" />
-        <child link="base_link" />
-    </joint>
     <link name="base_link">
         <visual>
@@ -55,12 +38,4 @@
             </material>
         </visual>
-         <surface>
-          <friction>
-            <ode>
-              <mu>12.0</mu>
-              <mu2>10.0</mu2>
-            </ode>
-          </friction>
-        </surface>
         <collision>
             <geometry>
@@ -80,12 +55,4 @@
             <material name="black"/>
         </visual>
-         <surface>
-          <friction>
-            <ode>
-              <mu>12.0</mu>
-              <mu2>10.0</mu2>
-            </ode>
-          </friction>
-        </surface>
         <collision>
             <geometry>
@@ -105,12 +72,4 @@
             <material name="black"/>
         </visual>
-         <!-- <surface>
-          <friction>
-            <ode>
-              <mu>5.0</mu>
-              <mu2>10.0</mu2>
-            </ode>
-          </friction>
-        </surface> -->
         <collision>
             <geometry>
@@ -130,12 +89,4 @@
             <material name="black"/>
         </visual>
-         <!-- <surface>
-          <friction>
-            <ode>
-              <mu>5.0</mu>
-              <mu2>10.0</mu2>
-            </ode>
-          </friction>
-        </surface> -->
         <collision>
             <geometry>
@@ -222,10 +173,13 @@
     <gazebo>
         <plugin name="mecanum_controller" filename="libgazebo_ros_planar_move.so">
-            <alwaysOn>true</alwaysOn>
-            <updateRate>20.0</updateRate>
-            <robotNamespace>/</robotNamespace>
-            <commandTopic>cmd_vel</commandTopic>
-            <odometryTopic>odom</odometryTopic>
-            <odometryFrame>odom</odometryFrame>
+            <ros>
+                <!-- <namespace>/demo</namespace> -->
+                <remapping>cmd_vel:=cmd_vel</remapping>
+                <remapping>odom:=odom</remapping>
+            </ros>
+            <update_rate>100</update_rate>
+            <publish_rate>100</publish_rate>
+            <publish_odom>false</publish_odom>
+            <publish_odom_tf>false</publish_odom_tf>
             <leftFrontJoint>base_to_wheel1</leftFrontJoint>
             <rightFrontJoint>base_to_wheel3</rightFrontJoint>
@@ -234,9 +188,4 @@
             <wheelSeparation>0.26</wheelSeparation>
             <wheelDiameter>0.12</wheelDiameter>
-            <odometryRate>20.0</odometryRate>
-            <torque>2</torque>
-            <robotBaseFrame>base_footprint</robotBaseFrame>
-            <publishOdomTF>true</publishOdomTF>
-            <broadcastTF>true</broadcastTF>
         </plugin>
     </gazebo>
@@ -251,5 +200,5 @@
             <topic>__default_topic__</topic>
             <plugin filename="libgazebo_ros_imu_sensor.so" name="imu_plugin">
-                <topicName>imu</topicName>
+                <topicName>/livox/imu</topicName>
                 <bodyName>imu_link</bodyName>
                 <updateRateHZ>100.0</updateRateHZ>
@@ -264,5 +213,5 @@
                 <randomWalk>0.0</randomWalk>
                 <ros>
-                    <remapping>~/out:=/imu</remapping>
+                    <remapping>~/out:=/livox/imu</remapping>
                 </ros>
             </plugin>
@@ -271,5 +220,5 @@
     <!-- Livox-Mid360  -->
     <xacro:include filename="$(find ros2_livox_simulation)/urdf/mid360.xacro" />
-    <xacro:mid360 name="livox" parent="base_link" topic="mid360">
+    <xacro:mid360 name="livox_frame" parent="base_link" topic="/livox/lidar">
         <origin xyz="0 0.0 0.175" rpy="0 0 0"/>
     </xacro:mid360>

Commit message: fixed imu data making pointcloud unseen, still don't the reason

File: rc_map/urdf/waking_robot.xacro (robot description, xacro)
@@ -11,4 +11,21 @@
         </inertial>
     </xacro:macro>
+    <link name="base_footprint">
+        <visual>
+            <geometry>
+                <box size="0.001 0.001 0.001"/>
+            </geometry>
+            <origin rpy="0 0 0" xyz="0 0 0"/>
+        </visual>
+    </link>
+    <gazebo reference="base_footprint">
+        <material>Gazebo/Green</material>
+        <turnGravityOff>false</turnGravityOff>
+    </gazebo>
+    <joint name="base_footprint_joint" type="fixed">
+        <origin xyz="0 0 0" />
+        <parent link="base_footprint" />
+        <child link="base_link" />
+    </joint>
     <link name="base_link">
         <visual>
@@ -38,4 +55,12 @@
             </material>
         </visual>
+         <surface>
+          <friction>
+            <ode>
+              <mu>12.0</mu>
+              <mu2>10.0</mu2>
+            </ode>
+          </friction>
+        </surface>
         <collision>
             <geometry>
@@ -55,4 +80,12 @@
             <material name="black"/>
         </visual>
+         <surface>
+          <friction>
+            <ode>
+              <mu>12.0</mu>
+              <mu2>10.0</mu2>
+            </ode>
+          </friction>
+        </surface>
         <collision>
             <geometry>
@@ -72,4 +105,12 @@
             <material name="black"/>
         </visual>
+         <!-- <surface>
+          <friction>
+            <ode>
+              <mu>5.0</mu>
+              <mu2>10.0</mu2>
+            </ode>
+          </friction>
+        </surface> -->
         <collision>
             <geometry>
@@ -89,4 +130,12 @@
             <material name="black"/>
         </visual>
+         <!-- <surface>
+          <friction>
+            <ode>
+              <mu>5.0</mu>
+              <mu2>10.0</mu2>
+            </ode>
+          </friction>
+        </surface> -->
         <collision>
             <geometry>
@@ -173,13 +222,10 @@
     <gazebo>
         <plugin name="mecanum_controller" filename="libgazebo_ros_planar_move.so">
-            <ros>
-                <!-- <namespace>/demo</namespace> -->
-                <remapping>cmd_vel:=cmd_vel</remapping>
-                <remapping>odom:=odom</remapping>
-            </ros>
-            <update_rate>100</update_rate>
-            <publish_rate>100</publish_rate>
-            <publish_odom>false</publish_odom>
-            <publish_odom_tf>false</publish_odom_tf>
+            <alwaysOn>true</alwaysOn>
+            <updateRate>20.0</updateRate>
+            <robotNamespace>/</robotNamespace>
+            <commandTopic>cmd_vel</commandTopic>
+            <odometryTopic>odom</odometryTopic>
+            <odometryFrame>odom</odometryFrame>
             <leftFrontJoint>base_to_wheel1</leftFrontJoint>
             <rightFrontJoint>base_to_wheel3</rightFrontJoint>
@@ -188,4 +234,9 @@
             <wheelSeparation>0.26</wheelSeparation>
             <wheelDiameter>0.12</wheelDiameter>
+            <odometryRate>20.0</odometryRate>
+            <torque>2</torque>
+            <robotBaseFrame>base_footprint</robotBaseFrame>
+            <publishOdomTF>true</publishOdomTF>
+            <broadcastTF>true</broadcastTF>
         </plugin>
     </gazebo>
@@ -200,5 +251,5 @@
             <topic>__default_topic__</topic>
             <plugin filename="libgazebo_ros_imu_sensor.so" name="imu_plugin">
-                <topicName>/livox/imu</topicName>
+                <topicName>imu</topicName>
                 <bodyName>imu_link</bodyName>
                 <updateRateHZ>100.0</updateRateHZ>
@@ -213,5 +264,5 @@
                 <randomWalk>0.0</randomWalk>
                 <ros>
-                    <remapping>~/out:=/livox/imu</remapping>
+                    <remapping>~/out:=/imu</remapping>
                 </ros>
             </plugin>
@@ -220,5 +271,5 @@
     <!-- Livox-Mid360  -->
     <xacro:include filename="$(find ros2_livox_simulation)/urdf/mid360.xacro" />
-    <xacro:mid360 name="livox_frame" parent="base_link" topic="/livox/lidar">
+    <xacro:mid360 name="livox" parent="base_link" topic="mid360">
         <origin xyz="0 0.0 0.175" rpy="0 0 0"/>
     </xacro:mid360>

Commit message: ADD online_async_launch
Signed-off-by: weison <weisonweileen@gmail.com>

File: rc_map/urdf/waking_robot.xacro (robot description, xacro)
@@ -11,21 +11,4 @@
         </inertial>
     </xacro:macro>
-    <link name="base_footprint">
-        <visual>
-            <geometry>
-                <box size="0.001 0.001 0.001"/>
-            </geometry>
-            <origin rpy="0 0 0" xyz="0 0 0"/>
-        </visual>
-    </link>
-    <gazebo reference="base_footprint">
-        <material>Gazebo/Green</material>
-        <turnGravityOff>false</turnGravityOff>
-    </gazebo>
-    <joint name="base_footprint_joint" type="fixed">
-        <origin xyz="0 0 0" />
-        <parent link="base_footprint" />
-        <child link="base_link" />
-    </joint>
     <link name="base_link">
         <visual>
@@ -42,4 +25,5 @@
                 <box size="0.2 .3 0.1"/>
             </geometry>
+            <origin rpy="0 0 ${PI/2}" xyz="0 0 0.05"/>
         </collision>
         <xacro:default_inertial mass="8.2"/>
@@ -55,12 +39,4 @@
             </material>
         </visual>
-         <surface>
-          <friction>
-            <ode>
-              <mu>12.0</mu>
-              <mu2>10.0</mu2>
-            </ode>
-          </friction>
-        </surface>
         <collision>
             <geometry>
@@ -80,12 +56,4 @@
             <material name="black"/>
         </visual>
-         <surface>
-          <friction>
-            <ode>
-              <mu>12.0</mu>
-              <mu2>10.0</mu2>
-            </ode>
-          </friction>
-        </surface>
         <collision>
             <geometry>
@@ -105,12 +73,4 @@
             <material name="black"/>
         </visual>
-         <!-- <surface>
-          <friction>
-            <ode>
-              <mu>5.0</mu>
-              <mu2>10.0</mu2>
-            </ode>
-          </friction>
-        </surface> -->
         <collision>
             <geometry>
@@ -130,12 +90,4 @@
             <material name="black"/>
         </visual>
-         <!-- <surface>
-          <friction>
-            <ode>
-              <mu>5.0</mu>
-              <mu2>10.0</mu2>
-            </ode>
-          </friction>
-        </surface> -->
         <collision>
             <geometry>
@@ -222,10 +174,13 @@
     <gazebo>
         <plugin name="mecanum_controller" filename="libgazebo_ros_planar_move.so">
-            <alwaysOn>true</alwaysOn>
-            <updateRate>20.0</updateRate>
-            <robotNamespace>/</robotNamespace>
-            <commandTopic>cmd_vel</commandTopic>
-            <odometryTopic>odom</odometryTopic>
-            <odometryFrame>odom</odometryFrame>
+            <ros>
+                <!-- <namespace>/demo</namespace> -->
+                <remapping>cmd_vel:=cmd_vel</remapping>
+                <remapping>odom:=odom</remapping>
+            </ros>
+            <update_rate>100</update_rate>
+            <publish_rate>100</publish_rate>
+            <publish_odom>false</publish_odom>
+            <publish_odom_tf>false</publish_odom_tf>
             <leftFrontJoint>base_to_wheel1</leftFrontJoint>
             <rightFrontJoint>base_to_wheel3</rightFrontJoint>
@@ -234,14 +189,9 @@
             <wheelSeparation>0.26</wheelSeparation>
             <wheelDiameter>0.12</wheelDiameter>
-            <odometryRate>20.0</odometryRate>
-            <torque>2</torque>
-            <robotBaseFrame>base_footprint</robotBaseFrame>
-            <publishOdomTF>true</publishOdomTF>
-            <broadcastTF>true</broadcastTF>
         </plugin>
     </gazebo>
     <!-- imu控制 -->
     <gazebo reference="imu_link">
-        <material>Gazebo/Orange</material>
+        <material>Gazebo/Blue</material>
         <gravity>true</gravity>
         <sensor name="imu_sensor" type="imu">
@@ -251,5 +201,5 @@
             <topic>__default_topic__</topic>
             <plugin filename="libgazebo_ros_imu_sensor.so" name="imu_plugin">
-                <topicName>imu</topicName>
+                <topicName>/livox/imu</topicName>
                 <bodyName>imu_link</bodyName>
                 <updateRateHZ>100.0</updateRateHZ>
@@ -264,5 +214,5 @@
                 <randomWalk>0.0</randomWalk>
                 <ros>
-                    <remapping>~/out:=/imu</remapping>
+                    <remapping>~/out:=/livox/imu</remapping>
                 </ros>
             </plugin>
@@ -271,5 +221,5 @@
     <!-- Livox-Mid360  -->
     <xacro:include filename="$(find ros2_livox_simulation)/urdf/mid360.xacro" />
-    <xacro:mid360 name="livox" parent="base_link" topic="mid360">
+    <xacro:mid360 name="livox_frame" parent="base_link" topic="/livox/lidar">
         <origin xyz="0 0.0 0.175" rpy="0 0 0"/>
     </xacro:mid360>
